Commit message: new urdf with more than one link

File: right-arm/robot.urdf (robot description, URDF)
Before this commit: robot onshape, 1 links, 0 joints
Links:
- removed link wbh_m2_5x10
- added link baseplaterev2, mass 0; collision mesh filename=package://.5_hexbearing_1.125_od.stl; collision mesh filename=package://.5_hexbearing_1.125_od.stl
- added link shoulderbaseplaterev2, mass 0; collision mesh filename=package://shoulderbaseplaterev2.stl; visual mesh filename=package://shoulderbaseplaterev2.stl
Joints:
- added joint part1: type revolute, parent baseplaterev2, child shoulderbaseplaterev2, origin xyz=-0.050972 -0.0908091 -0.0376234 rpy=-3.14159 -1.92382e-16 2.15452, axis 0 0 1, limit effort=1 velocity=20

Commit message: created new urdf file

File: right-arm/robot.urdf (robot description, URDF)
Before this commit: robot onshape, 2 links, 1 joints
Links:
- removed link baseplaterev2
- removed link shoulderbaseplaterev2
- added link link_base_link, mass 0; collision mesh filename=package://.5_hexbearing_1.125_od.stl; collision mesh filename=package://.5_hexbearing_1.125_od.stl
- added link link_claw, mass 0; collision mesh filename=package://dc12_a01_spacer_ring.stl; collision mesh filename=package://dc12_a01_spacer_ring.stl
- added link link_elbow, mass 0; collision mesh filename=package://10-32_x_0.75in_buttonhead_locking_screw_mcmaster_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; collision mesh filename=package://10-32_x_0.75in_buttonhead_locking_screw_mcmaster_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
- added link link_forearm, mass 0; collision mesh filename=package://10-32_x_0.75in_buttonhead_locking_screw_mcmaster_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; collision mesh filename=package://10-32_x_0.75in_buttonhead_locking_screw_mcmaster_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
- added link link_socket, mass 0; collision mesh filename=package://.5_hexbearing_1.125_od.stl; collision mesh filename=package://.5_hexbearing_1.125_od.stl
Joints:
- added joint part2: type revolute, parent link_elbow, child link_socket, origin xyz=9.71445e-17 -0.181143 -0.0251898 rpy=8.61858e-16 -8.14474e-16 -0.340595, axis 0 0 1, limit effort=1 velocity=20
- added joint part3: type revolute, parent link_forearm, child link_elbow, origin xyz=0.0215451 -0.081375 0.226287 rpy=1.5708 0.269717 0.979301, axis 0 0 1, limit effort=1 velocity=20
- added joint part4: type revolute, parent link_forearm, child link_claw, origin xyz=0.0168036 -0.034632 0.401022 rpy=-2.93853 0.0201748 2.45243, axis 0 0 1, limit effort=1 velocity=20
- joint part1: child shoulderbaseplaterev2 -> link_base_link; origin xyz=-0.050972 -0.0908091 -0.0376234 rpy=-3.14159 -1.92382e-16 2.15452 -> xyz=0.0511893 -0.073192 -0.0297467 rpy=-0.960485 -1.5708 0; parent baseplaterev2 -> link_socket

Commit message: added new good urdf after reordering mates

File: right-arm/robot.urdf (robot description, URDF)
Before this commit: robot onshape, 5 links, 4 joints
Joints:
- joint part1: child link_base_link -> link_socket; origin xyz=0.0511893 -0.073192 -0.0297467 rpy=-0.960485 -1.5708 0 -> xyz=-0.050972 -0.0908091 -0.0376234 rpy=3.14159 -4.29356e-16 2.5501; parent link_socket -> link_base_link
- joint part2: child link_socket -> link_elbow; origin xyz=9.71445e-17 -0.181143 -0.0251898 rpy=8.61858e-16 -8.14474e-16 -0.340595 -> xyz=-0.0297467 -2.91434e-16 -0.0893164 rpy=1.5708 0.960485 1.5708; parent link_elbow -> link_socket
- joint part3: child link_elbow -> link_forearm; origin xyz=0.0215451 -0.081375 0.226287 rpy=1.5708 0.269717 0.979301 -> xyz=0.166399 -0.0715838 -0.0251898 rpy=-1.66708e-14 -1.48395e-14 1.16453; parent link_forearm -> link_elbow
- joint part4: origin xyz=0.0168036 -0.034632 0.401022 rpy=-2.93853 0.0201748 2.45243 -> xyz=4.16334e-16 -0.178438 0.03 rpy=-1.5708 1.5708 0
